File: cece-pcb/cece-pcb.sch (KiCad schematic (older format))
At the start: 26 parts, among them J101 Li-Ion Battery, J102 SERIAL, J103 HTU21D, J104 VAC, K101 SANYOU_SRD_Form_C, Q101 Q_NPN, U101 TLV75533PDBV, U102 MCP73811T-420I-OT

Commit message: Boards have arrived. Fixed the many mistakes in the schematic
Parts:
- J103: renamed from J102; footprint Connector_PinHeader_2.54mm:PinHeader_1x05_P2.54mm_Vertical -> Connector_PinHeader_2.54mm:PinHeader_1x04_P2.54mm_Vertical; symbol Connector:Conn_01x05_Male -> Connector:Conn_01x04_Male
- renumbered C103 to C101, C101 to C102, C102 to C103, D102 to D101, D103 to D102, D101 to D103, J104 to J101, J103 to J102, J101 to J104, JP102 to JP101, JP101 to JP102, R104 to R101, R101 to R102, R105 to R103, R103 to R104, R102 to R105
Connections:
- net DTR is gone; now on net RX: J103.2 (Pin_2)
- net GND: now also J103.4 (Pin_4); no longer J103.5 (Pin_5)
- net RX: no longer J103.3 (Pin_3)
- net TX: now also J103.3 (Pin_3); no longer J103.4 (Pin_4)
- no-connect marks 5 -> 0
