File: cece-pcb/cece-pcb.sch (KiCad schematic (older format))
At the start: 26 parts, among them J101 VAC, J102 HTU21D, J103 SERIAL, J104 Li-Ion Battery, K101 SANYOU_SRD_Form_C, Q101 Q_NPN, U101 TLV75533PDBV, U102 MCP73811T-420I-OT

Commit message: Add diode to protect the seral input when 3V3 are already supplied internally and shuffle stuff around a bit on the layout
Parts:
- removed R102: 12_DNP, Resistor_THT:R_Axial_DIN0207_L6.3mm_D2.5mm_P7.62mm_Horizontal, symbol Device:R_US
- added D104: Schottky SOT-23, Diode_SMD:D_SOT-23_ANK, symbol Device:D_Schottky
- added D105: Schottky SOD-123, Diode_SMD:D_SOD-123F, symbol Device:D_Schottky
- added JP103: 73811, Jumper:SolderJumper-2_P1.3mm_Open_Pad1.0x1.5mm, symbol Jumper:SolderJumper_2_Open
- R105: footprint Resistor_THT:R_Axial_DIN0207_L6.3mm_D2.5mm_P7.62mm_Horizontal -> Resistor_SMD:R_0805_2012Metric_Pad1.15x1.40mm_HandSolder
Connections:
- net +3V3: now also D104.1 (K), D105.1 (K); no longer J103.1 (Pin_1)
- net +5V: now also JP103.1 (A)
- net at R105.1, U102.5 (PROG): now also JP103.2 (B)
- new net: D104.2 (A), D105.2 (A), J103.1 (Pin_1)
Other:
- moved on the sheet: J103
Changed lines of the file:
@@
 L Connector:Conn_01x04_Male J103
 U 1 1 5FD6FD7F
-P 5400 2850
-F 0 "J103" H 5372 2782 50  0000 R CNN
-F 1 "SERIAL" H 5372 2873 50  0000 R CNN
-F 2 "Connector_PinHeader_2.54mm:PinHeader_1x04_P2.54mm_Vertical" H 5400 2850 50  0001 C CNN
-F 3 "~" H 5400 2850 50  0001 C CNN
-	1    5400 2850
+P 5250 2200
+F 0 "J103" H 5222 2132 50  0000 R CNN
+F 1 "SERIAL" H 5222 2223 50  0000 R CNN
+F 2 "Connector_PinHeader_2.54mm:PinHeader_1x04_P2.54mm_Vertical" H 5250 2200 50  0001 C CNN
+F 3 "~" H 5250 2200 50  0001 C CNN
+	1    5250 2200
 	-1   0    0    1
 $EndComp
 Wire Wire Line
-	5050 2750 5200 2750
-Wire Wire Line
-	5200 2850 5050 2850
+	4900 2100 5050 2100
+Wire Wire Line
+	5050 2200 4900 2200
 $Comp
 L power:GND #PWR0104
 U 1 1 5FD73334
-P 4900 2650
-F 0 "#PWR0104" H 4900 2400 50  0001 C CNN
-F 1 "GND" H 4905 2477 50  0000 C CNN
-F 2 "" H 4900 2650 50  0001 C CNN
-F 3 "" H 4900 2650 50  0001 C CNN
-	1    4900 2650
-	1    0    0    -1
-$EndComp
-Text Label 5050 2750 0    50   ~ 0
+P 4750 1900
+F 0 "#PWR0104" H 4750 1650 50  0001 C CNN
+F 1 "GND" H 4755 1727 50  0000 C CNN
+F 2 "" H 4750 1900 50  0001 C CNN
+F 3 "" H 4750 1900 50  0001 C CNN
+	1    4750 1900
+	1    0    0    -1
+$EndComp
+Text Label 4900 2100 0    50   ~ 0
 TX
-Text Label 5050 2850 0    50   ~ 0
+Text Label 4900 2200 0    50   ~ 0
 RX
 $Comp
@@
 Connection ~ 2000 4350
 $Comp
-L Device:R_US R102
-U 1 1 5FDCA40C
-P 1250 4600
-F 0 "R102" H 1318 4646 50  0000 L CNN
-F 1 "12_DNP" H 1318 4555 50  0000 L CNN
-F 2 "Resistor_THT:R_Axial_DIN0207_L6.3mm_D2.5mm_P7.62mm_Horizontal" V 1290 4590 50  0001 C CNN
-F 3 "~" H 1250 4600 50  0001 C CNN
-	1    1250 4600
-	1    0    0    -1
-$EndComp
-$Comp
 L Device:R_US R105
 U 1 1 5FDCAD59
@@
 F 0 "R105" H 1318 5046 50  0000 L CNN
 F 1 "R_PROG" H 1318 4955 50  0000 L CNN
-F 2 "Resistor_THT:R_Axial_DIN0207_L6.3mm_D2.5mm_P7.62mm_Horizontal" V 1290 4990 50  0001 C CNN
+F 2 "Resistor_SMD:R_0805_2012Metric_Pad1.15x1.40mm_HandSolder" V 1290 4990 50  0001 C CNN
 F 3 "~" H 1250 5000 50  0001 C CNN
 	1    1250 5000
@@
 $EndComp
 Wire Wire Line
-	4900 2650 5200 2650
-Wire Wire Line
 	9900 2900 10000 2900
 Wire Wire Line
@@
 Wire Wire Line
 	2550 4350 2450 4350
-Wire Wire Line
-	4650 2950 5200 2950
 $Comp
 L power:+3V3 #PWR0108
 U 1 1 5FD72E0B
-P 4650 2950
-F 0 "#PWR0108" H 4650 2800 50  0001 C CNN
-F 1 "+3V3" H 4665 3123 50  0000 C CNN
-F 2 "" H 4650 2950 50  0001 C CNN
-F 3 "" H 4650 2950 50  0001 C CNN
-	1    4650 2950
-	1    0    0    -1
+P 4500 2300
+F 0 "#PWR0108" H 4500 2150 50  0001 C CNN
+F 1 "+3V3" H 4515 2473 50  0000 C CNN
+F 2 "" H 4500 2300 50  0001 C CNN
+F 3 "" H 4500 2300 50  0001 C CNN
+	1    4500 2300
+	1    0    0    -1
+$EndComp
+$Comp
+L Device:D_Schottky D104
+U 1 1 6026BD54
+P 4800 2350
+F 0 "D104" H 4800 2150 50  0000 C CNN
+F 1 "Schottky SOT-23" H 4800 2250 50  0000 C CNN
+F 2 "Diode_SMD:D_SOT-23_ANK" H 4800 2350 50  0001 C CNN
+F 3 "~" H 4800 2350 50  0001 C CNN
+	1    4800 2350
+	1    0    0    -1
+$EndComp
+Wire Wire Line
+	5050 2300 5000 2300
+Wire Wire Line
+	5000 2300 5000 2350
+Wire Wire Line
+	5000 2350 4950 2350
+Wire Wire Line
+	4650 2350 4600 2350
+Wire Wire Line
+	4500 2350 4500 2300
+Wire Wire Line
+	4750 1900 4750 1850
+Wire Wire Line
+	5000 1850 5000 2000
+Wire Wire Line
+	5000 2000 5050 2000
+Wire Wire Line
+	4750 1850 5000 1850
+$Comp
+L Device:D_Schottky D105
+U 1 1 6027D132
+P 4800 2650
+F 0 "D105" H 4800 2450 50  0000 C CNN
+F 1 "Schottky SOD-123" H 4800 2550 50  0000 C CNN
+F 2 "Diode_SMD:D_SOD-123F" H 4800 2650 50  0001 C CNN
+F 3 "~" H 4800 2650 50  0001 C CNN
+	1    4800 2650
+	1    0    0    -1
+$EndComp
+Wire Wire Line
+	5000 2350 5000 2650
+Wire Wire Line
+	5000 2650 4950 2650
+Connection ~ 5000 2350
+Wire Wire Line
+	4650 2650 4600 2650
+Wire Wire Line
+	4600 2650 4600 2350
+Connection ~ 4600 2350
+Wire Wire Line
+	4600 2350 4500 2350
+$Comp
+L Jumper:SolderJumper_2_Open JP103
+U 1 1 602D11B4
+P 1250 4600
+F 0 "JP103" H 1250 4805 50  0000 C CNN
+F 1 "73811" H 1250 4714 50  0000 C CNN
+F 2 "Jumper:SolderJumper-2_P1.3mm_Open_Pad1.0x1.5mm" H 1250 4600 50  0001 C CNN
+F 3 "~" H 1250 4600 50  0001 C CNN
+	1    1250 4600
+	0    1    1    0
 $EndComp
 $EndSCHEMATC

Commit message: Use new stuff from pol lib
Parts:
- added EA101: a_black_cat, pol:a_black_cat, symbol pol:a_black_cat
Changed lines of the file:
@@
 	0    1    1    0
 $EndComp
+$Comp
+L pol:a_black_cat EA101
+U 1 1 605E1AB3
+P 7450 6850
+F 0 "EA101" H 8090 6865 50  0000 L CNN
+F 1 "a_black_cat" H 8090 6774 50  0000 L CNN
+F 2 "pol:a_black_cat" H 7450 6850 50  0001 C CNN
+F 3 "" H 7450 6850 50  0001 C CNN
+	1    7450 6850
+	1    0    0    -1
+$EndComp
 $EndSCHEMATC
